Commit message: Add files via upload

File: urdf/sensors/rplidar.urdf.xacro (robot description, xacro)
@@ -18,5 +18,5 @@
           <geometry>
           <mesh filename="package://hector_sensors_description/meshes/hokuyo_utm30lx/hokuyo_utm_30lx$(optenv TEST_SELF_FILTER).dae"/>
-        </geometry>
+	</geometry>
         </visual>
         <collision>
